File: ZTL-Badge-Hardware.kicad_pcb (KiCad board)
At the start: 2 copper layers, 17 parts, among them J1 UART, J2 ISP, J3 External Power Supply, SW1 Left Button, SW2 Right Button, SW3 Power Switch, U1 ATmega328P-P, Y1 8MHz

Commit message: first layout
Parts:
- removed J3: External Power Supply, Connector_PinHeader_2.54mm:PinHeader_1x02_P2.54mm_Vertical
- BT1: moved to B.Cu
- H1: footprint MountingHole:MountingHole_5.3mm_M5_DIN965 -> MountingHole:MountingHole_5.3mm_M5_DIN965_Pad
- moved J2 112.9 mm to (166.0, 119.5)
- moved U1 103.3 mm to (123.5, 126.0), turned to 90 degrees
- moved SW1 86.5 mm to (176.0, 97.5), turned to 90 degrees
- moved J1 78.7 mm to (146.3, 139.5), turned to -90 degrees
- moved Y1 75.2 mm to (146.9, 134.5), turned to 180 degrees
- moved D1 67.1 mm to (140.0, 97.5), turned to 90 degrees
- moved SW3 62.3 mm to (117.0, 142.0), turned to 180 degrees
- moved C1 59.7 mm to (128.5, 135.8), turned to -90 degrees
- moved C3 56.4 mm to (146.2, 129.0)
- moved C2 54.6 mm to (138.2, 129.0), turned to 180 degrees
- moved C4 51.5 mm to (143.5, 129.0), turned to 180 degrees
- moved R1 44.7 mm to (123.5, 130.7), turned to -90 degrees
- moved SW2 43.0 mm to (104.0, 97.5), turned to 90 degrees
- moved BT1 41.4 mm to (110.0, 116.4), turned to -90 degrees
- moved C5 36.6 mm to (117.0, 133.2), turned to 90 degrees
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Connections:
- J1 pad 3: +3V0 -> POWER_IN
- SW3 pad 1: Net-(J3-Pin_1) -> POWER_IN
Routing:
- net +3V0: track 0.00 -> 103.5 mm
- net Net-(J2-Pin_4): track 0.00 -> 81.1 mm
- net RESET: track 0.00 -> 53.9 mm
- net LED_Y6: track 0.00 -> 53.2 mm, vias 0 -> 1
- net LED_X2: track 0.00 -> 51.3 mm
- net LED_Y7: track 0.00 -> 50.9 mm, vias 0 -> 1
- net LED_Y4: track 0.00 -> 47.9 mm, vias 0 -> 1
- net LED_X3: track 0.00 -> 47.6 mm, vias 0 -> 1
- net LED_X5: track 0.00 -> 42.9 mm
- net LED_Y2: track 0.00 -> 41.1 mm, vias 0 -> 1
- net LED_X0: track 0.00 -> 40.4 mm
- net Net-(U1-PB2): track 0.00 -> 39.0 mm
- net Net-(BT1-+): track 0.00 -> 37.8 mm
- net LED_Y1: track 0.00 -> 33.6 mm, vias 0 -> 1
- net LED_X1: track 0.00 -> 31.8 mm, vias 0 -> 1
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- added copper zone on B.Cu, net GND
- added copper zone on F.Cu, net GND
Other:
- board outline added: 80 x 80 mm
- board text added: "AN"
- board text added: "AUS"
- board text added: "DTR"
- board text added: "GND"
- board text added: "ISP"
- board text added: "RX"
- board text added: "TX"
- board text added: "VCC"
- board text added: "ZTL-Badge 2024 v1.0"
