File: ZTL-Badge-Hardware.kicad_sch (KiCad schematic)
At the start: 17 parts, among them J1 UART, J2 ISP, J3 External Power Supply, SW1 Left Button, SW2 Right Button, SW3 Power Switch, U1 ATmega328P-P, Y1 8MHz

Commit message: first layout
Parts:
- removed J3: External Power Supply, Connector_PinHeader_2.54mm:PinHeader_1x02_P2.54mm_Vertical, symbol Connector_Generic:Conn_01x02
- H1: footprint MountingHole:MountingHole_5.3mm_M5_DIN965 -> MountingHole:MountingHole_5.3mm_M5_DIN965_Pad
Connections:
- net +3V0: no longer J1.3 (Pin_3)
- net POWER_IN: now reaches SW3.1 (A)
- net POWER_IN: now also J1.3 (Pin_3)
Other:
- moved on the sheet: J1
